File: VideoModCCE/VideoModCCE.kicad_pcb (KiCad board)
At the start: 2 copper layers, 35 x 31.2 mm, 15 parts, among them Q1 BC558, Q2 BC548

Commit message: PCB Schematic Fix
Connections:
- C1 pad 1: Net-(C1-Pad1) -> Net-(Q2-Pad1)
- PIN3 pad 1: Net-(C1-Pad1) -> Net-(Q2-Pad1)
- R1 pad 2: Net-(C1-Pad1) -> Net-(R1-Pad2)
- R2 pad 1: Net-(C1-Pad1) -> Net-(R1-Pad2)
- R3 pad 1: Net-(C1-Pad1) -> Net-(R1-Pad2)
Routing:
- net Net-(Q2-Pad1): track 21.0 -> 44.5 mm
- net Net-(C1-Pad1): track 18.7 -> 0.00 mm
- net Net-(R1-Pad2): track 0.00 -> 7.00 mm
- net Net-(Q2-Pad2): track 20.6 -> 19.3 mm
