File: VideoModCCE/VideoModCCE.kicad_sch (KiCad schematic)
At the start: 14 parts

Commit message: PCB Schematic Fix
Parts:
- C1: value (none) -> 1uF; footprint (none) -> Capacitor_THT:C_Disc_D4.3mm_W1.9mm_P5.00mm
- C2: value (none) -> 100uF 16V; footprint (none) -> Capacitor_THT:CP_Radial_D8.0mm_P3.50mm
- PIN1: value (none) -> GND; footprint (none) -> TestPoint:TestPoint_Pad_3.0x3.0mm
- PIN2: value (none) -> CVBS IN; footprint (none) -> TestPoint:TestPoint_Pad_3.0x3.0mm
- PIN3: value (none) -> +5V; footprint (none) -> TestPoint:TestPoint_Pad_3.0x3.0mm
- PIN4: value (none) -> CVBS OUT; footprint (none) -> TestPoint:TestPoint_Pad_3.0x3.0mm
- Q1: value (none) -> BC558; footprint (none) -> Package_TO_SOT_THT:TO-92_HandSolder
- Q2: value (none) -> BC548; footprint (none) -> Package_TO_SOT_THT:TO-92_HandSolder
- R1: value (none) -> 220R; footprint (none) -> Resistor_THT:R_Axial_DIN0207_L6.3mm_D2.5mm_P7.62mm_Horizontal
- R2: value (none) -> 2K2; footprint (none) -> Resistor_THT:R_Axial_DIN0207_L6.3mm_D2.5mm_P7.62mm_Horizontal
- R3: value (none) -> 470R; footprint (none) -> Resistor_THT:R_Axial_DIN0207_L6.3mm_D2.5mm_P7.62mm_Horizontal
- R4: value (none) -> 75R; footprint (none) -> Resistor_THT:R_Axial_DIN0207_L6.3mm_D2.5mm_P7.62mm_Horizontal
- R5: value (none) -> 150R; footprint (none) -> Resistor_THT:R_Axial_DIN0207_L6.3mm_D2.5mm_P7.62mm_Horizontal
Connections:
- net at R1.2, R2.1, R3.1: no longer C1.1, PIN3.1
- net at Q2.1 (C), R2.2: now also C1.1, PIN3.1
Other:
- moved on the sheet: C1, PIN3
